File: Audio_Dac_I2S/Audio_Dac_I2S.sch (KiCad schematic (older format))
At the start: 35 parts

Commit message: making progress on PCB
Parts:
- added J?: AVR-JTAG-10, symbol Connector:AVR-JTAG-10
Connections:
- net labels added: NC, V1, V2, V3, V4, VCC_JTAG, tck, tdi, tdo, tms
- wire segments 80 -> 321
Other:
- moved on the sheet: A, B, C, D, E, F, G, H, J, K, M, N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

Commit message: made schematic updates
Parts:
- removed A: Conn_01x18, symbol Connector_Generic:Conn_01x18
- added R? (x6): 10K, symbol Device:R
Connections:
- net labels added: V1.2, V3.3, VCCIO, VCCIO_B8
- net labels removed: NC, V1
- wire segments 321 -> 245
- no-connect marks 0 -> 3

Commit message: editted fpga symbol and made jtag footprint
Parts:
- removed B, C, D, E, F, G, H, J, K, L, M, N, P, R, T, U, V: Conn_01x18, symbol Connector_Generic:Conn_01x18
- added J? (x10): Conn_01x20_Male, symbol Connector:Conn_01x20_Male
- added J?: Conn_01x09_Male, symbol Connector:Conn_01x09_Male
- added J?: Conn_01x17_Male, symbol Connector:Conn_01x17_Male
Connections:
- net labels removed: V1.2, V2, V3, V4, VCCIO
- wire segments 245 -> 299
- no-connect marks 3 -> 101
Other:
- moved on the sheet: IC?, J?, R?

Commit message: hopefully finished schematic
Parts:
- removed U?: FPGA, symbol CustomLib:FPGA
- added C? (x4): 10pF, symbol Device:C
- added D? (x4): DIODE, symbol pspice:DIODE
- added R?: 10K, symbol Device:R
- added clk?: tco-711AR, symbol CustomLib:tco-711AR
Connections:
- net VCC_JTAG is gone; now on net V3.3: J?.17 (3V3)
- net GND: now also J?.14 (GND), J?.20 (GND), J?.25 (GND), J?.30 (GND), J?.34 (GND), J?.39 (GND), J?.6 (GND), J?.9 (GND), C?.2, C?.2, C?.2, C?.2, R?.2, clk?.2 (GND); no longer U?.2 (DEM/SCLK)
- net V3.3: now also D?.2 (A), D?.2 (A), D?.2 (A), D?.2 (A), clk?.4 (VCC); no longer IC?.G8 (IO_48), IC?.H8 (IO_63), R?.1, R?.1
- net tck: now also C?.1, D?.1 (K)
- net tdi: now also C?.1, D?.1 (K)
- net tdo: now also C?.1, D?.1 (K)
- net tms: now also C?.1, D?.1 (K)
- net SDATA: now reaches U?.1 (SDATA)
- net SDATA: now also IC?.A6 (IO_5), J?.6 (Pin_6)
- net LRCK: now reaches U?.3 (LRCK)
- net LRCK: now also IC?.A8 (IO_6), J?.7 (Pin_7)
- net MCLK: now reaches U?.4 (MCLK)
- net MCLK: now also IC?.A9 (IO_7), J?.8 (Pin_8)
- net DATA: now reaches J?.40 (GPIO21/SCLK1)
- net DATA: now also IC?.A3 (IO_2), J?.3 (Pin_3)
- net INTERR: now reaches J?.18 (GPIO24)
- net INTERR: now also IC?.A4 (IO_3), J?.4 (Pin_4)
- net EN: now reaches J?.16 (GPIO23)
- net EN: now also IC?.A5 (IO_4), J?.5 (Pin_5)
- net DCLK: now reaches J?.22 (GPIO25)
- net DCLK: now also IC?.A2 (IO_1), J?.2 (Pin_2)
- net CLK: now reaches IC?.M3 (IO_100), J?.17 (Pin_17)
- net CLK: now also clk?.3 (CLK_OUT)
- new net: R?.1, U?.2 (DEM/SCLK)
- new net: IC?.G8 (IO_48), R?.1
- new net: IC?.H8 (IO_63), R?.1
- no-connect marks 101 -> 102
Other:
- moved on the sheet: J?

Commit message: laying out the PCB
Parts:
- C1, C10, C2, C3, C4, C5, C6, C7, C8, C9: renamed from C?; footprint (none) -> Capacitor_THT:C_Rect_L7.0mm_W2.0mm_P5.00mm
- D1, D2, D3, D4: renamed from D?; footprint (none) -> Diode_THT:D_A-405_P7.62mm_Horizontal
- IC1: renamed from IC?; footprint BGA324C80P18X18_1500X1500X155 -> MyFootprints:BGA324C80P18X18_1500X1500X155
- J1: renamed from J?; footprint (none) -> MyFootprints:Raspberry_Pi_40_pin_socket
- J10, J11, J12, J2, J3, J4, J5, J6, J8, J9: renamed from J?; footprint (none) -> Connector_PinHeader_2.54mm:PinHeader_1x20_P2.54mm_Vertical
- J13: renamed from J?; footprint (none) -> Connector_PinHeader_2.54mm:PinHeader_1x17_P2.54mm_Vertical
- J14: renamed from J?; footprint (none) -> MyFootprints:Jtag_header
- J7: renamed from J?; footprint (none) -> Connector_PinHeader_2.54mm:PinHeader_1x09_P2.54mm_Vertical
- R1, R10, R11, R12, R13, R2, R3, R4, R5, R6, R7, R8, R9: renamed from R?; footprint (none) -> Resistor_THT:R_Axial_DIN0204_L3.6mm_D1.6mm_P7.62mm_Horizontal
- U1: renamed from U?; footprint (none) -> MyFootprints:DAC
- U2: renamed from U?; footprint (none) -> MyFootprints:Audio_Jack
- clk1: renamed from clk?; footprint (none) -> MyFootprints:tco-711
Connections:
- net GND: now also C3.1, C5.1

Commit message: Done
Parts:
- removed J10, J11, J12, J2, J4, J5, J6, J8, J9: Conn_01x20_Male, Connector_PinHeader_2.54mm:PinHeader_1x20_P2.54mm_Vertical, symbol Connector:Conn_01x20_Male
- removed J13: Conn_01x17_Male, Connector_PinHeader_2.54mm:PinHeader_1x17_P2.54mm_Vertical, symbol Connector:Conn_01x17_Male
- removed J7: Conn_01x09_Male, Connector_PinHeader_2.54mm:PinHeader_1x09_P2.54mm_Vertical, symbol Connector:Conn_01x09_Male
- removed R5: 10K, Resistor_THT:R_Axial_DIN0204_L3.6mm_D1.6mm_P7.62mm_Horizontal, symbol Device:R
- added DBG1: Conn_01x05_Male, Connector_PinHeader_2.54mm:PinHeader_1x05_P2.54mm_Vertical, symbol Connector:Conn_01x05_Male
- added J2: Conn_01x11_Male, Connector_PinHeader_2.54mm:PinHeader_1x11_P2.54mm_Vertical, symbol Connector:Conn_01x11_Male
- added PI_OUT1: Conn_01x04_Male, Connector_PinHeader_2.54mm:PinHeader_1x04_P2.54mm_Vertical, symbol Connector:Conn_01x04_Male
Connections:
- net labels added: a1, c10, c17, c18, c5, c6, c7, c8, c9, d15, d16, d17, d18, d4, d5, d6, d7, d8, e4, e5, h1, j1, k1, l1, m1, n1, p1, r1, u1, v1
- wire segments 283 -> 288
